Commit message: Update gazebo_control.xacro

File: description/gazebo_control.xacro (robot description, xacro)
@@ -12,5 +12,4 @@
             <state_interface name="position"/>
             <state_interface name="velocity"/>
-            <state_interface name="effort"/>
         </joint>
         <joint name="joint_xy">
@@ -21,5 +20,4 @@
             <state_interface name="position"/> <!--what i want to broadcast-->
             <state_interface name="velocity"/>
-            <state_interface name="effort"/>
         </joint>
         <joint name="joint_needle">
@@ -30,7 +28,6 @@
             <state_interface name="position"/>
             <state_interface name="velocity"/>
-            <state_interface name="effort"/>
         </joint>
-        <!--joint name="joint_${id}_x">
+        <joint name="joint_2_x">
             <command_interface name="position">
                 <param name="min">-3</param>
@@ -39,7 +36,6 @@
             <state_interface name="position"/>
             <state_interface name="velocity"/>
-            <state_interface name="effort"/>
         </joint>
-        <joint name="joint_${id}_y">
+        <joint name="joint_2_z">
             <command_interface name="position">
                 <param name="min">-3</param>
@@ -48,10 +44,57 @@
             <state_interface name="position"/>
             <state_interface name="velocity"/>
-            <state_interface name="effort"/>
-        </joint-->
+        </joint>
+        <joint name="joint_3_x">
+            <command_interface name="position">
+                <param name="min">-3</param>
+                <param name="max">3</param>
+            </command_interface>
+            <state_interface name="position"/>
+            <state_interface name="velocity"/>
+        </joint>
+        <joint name="joint_3_z">
+            <command_interface name="position">
+                <param name="min">-3</param>
+                <param name="max">3</param>
+            </command_interface>
+            <state_interface name="position"/>
+            <state_interface name="velocity"/>
+        </joint>
+        <joint name="joint_4_x">
+            <command_interface name="position">
+                <param name="min">-3</param>
+                <param name="max">3</param>
+            </command_interface>
+            <state_interface name="position"/>
+            <state_interface name="velocity"/>
+        </joint>
+        <joint name="joint_4_z">
+            <command_interface name="position">
+                <param name="min">-3</param>
+                <param name="max">3</param>
+            </command_interface>
+            <state_interface name="position"/>
+            <state_interface name="velocity"/>
+        </joint>
+        <joint name="joint_5_x">
+            <command_interface name="position">
+                <param name="min">-3</param>
+                <param name="max">3</param>
+            </command_interface>
+            <state_interface name="position"/>
+            <state_interface name="velocity"/>
+        </joint>
+        <joint name="joint_5_z">
+            <command_interface name="position">
+                <param name="min">-3</param>
+                <param name="max">3</param>
+            </command_interface>
+            <state_interface name="position"/>
+            <state_interface name="velocity"/>
+        </joint>
     </ros2_control>
     <gazebo>
         <plugin filename="libgazebo_ros2_control.so" name="gazebo_ros2_control">
-            <parameters>$(my_bot)/config/controller.yaml</parameters>
+            <parameters>$(find my_bot)/config/controller.yaml</parameters>
         </plugin>
     </gazebo>

Commit message: gazebo sim is working but pb with friction and weights, effort, velocity, upper qnd lower limits, radis and needle size

File: description/gazebo_control.xacro (robot description, xacro)
@@ -29,5 +29,5 @@
             <state_interface name="velocity"/>
         </joint>
-        <joint name="joint_2_x">
+        <joint name="link_2_aux_joint">
             <command_interface name="position">
                 <param name="min">-3</param>
@@ -37,5 +37,5 @@
             <state_interface name="velocity"/>
         </joint>
-        <joint name="joint_2_z">
+        <joint name="link_2_joint">
             <command_interface name="position">
                 <param name="min">-3</param>
@@ -45,5 +45,5 @@
             <state_interface name="velocity"/>
         </joint>
-        <joint name="joint_3_x">
+        <joint name="link_3_aux_joint">
             <command_interface name="position">
                 <param name="min">-3</param>
@@ -53,5 +53,5 @@
             <state_interface name="velocity"/>
         </joint>
-        <joint name="joint_3_z">
+        <joint name="link_3_joint">
             <command_interface name="position">
                 <param name="min">-3</param>
@@ -61,5 +61,5 @@
             <state_interface name="velocity"/>
         </joint>
-        <joint name="joint_4_x">
+        <joint name="link_4_aux_joint">
             <command_interface name="position">
                 <param name="min">-3</param>
@@ -69,5 +69,5 @@
             <state_interface name="velocity"/>
         </joint>
-        <joint name="joint_4_z">
+        <joint name="link_4_joint">
             <command_interface name="position">
                 <param name="min">-3</param>
@@ -77,5 +77,5 @@
             <state_interface name="velocity"/>
         </joint>
-        <joint name="joint_5_x">
+        <joint name="link_5_aux_joint">
             <command_interface name="position">
                 <param name="min">-3</param>
@@ -85,5 +85,5 @@
             <state_interface name="velocity"/>
         </joint>
-        <joint name="joint_5_z">
+        <joint name="link_5_joint">
             <command_interface name="position">
                 <param name="min">-3</param>

File: description/gazebo_tags.xacro (robot description, xacro)
@@ -9,12 +9,4 @@
         </xacro:if>
     </xacro:macro>
-    <xacro:macro name="add_gazebo_links" params="current_id max_id">
-        <xacro:if value="${current_id != max_id}">
-            <gazebo reference="link_${current_id}">
-                <material>Gazebo/Blue</material>
-            </gazebo>
-            <xacro:add_gazebo_links current_id="${current_id + 1}" max_id="${max_id}"/>
-        </xacro:if>
-    </xacro:macro>
     <gazebo>
         <plugin name="gazebo_ros_joint_state_publisher" filename="libgazebo_ros_joint_state_publisher.so">
@@ -23,12 +15,12 @@
             <joint_name>joint_zx</joint_name>
             <joint_name>joint_needle</joint_name>
-            <joint_name>joint_2_x</joint_name>
-            <joint_name>joint_3_x</joint_name>
-            <joint_name>joint_4_x</joint_name>
-            <joint_name>joint_5_x</joint_name>
-            <joint_name>joint_2_z</joint_name>
-            <joint_name>joint_3_z</joint_name>
-            <joint_name>joint_4_z</joint_name>
-            <joint_name>joint_5_z</joint_name>
+            <joint_name>link_2_aux_joint</joint_name>
+            <joint_name>link_3_aux_joint</joint_name>
+            <joint_name>link_4_aux_joint</joint_name>
+            <joint_name>link_5_aux_joint</joint_name>
+            <joint_name>link_2_joint</joint_name>
+            <joint_name>link_3_joint</joint_name>
+            <joint_name>link_4_joint</joint_name>
+            <joint_name>link_5_joint</joint_name>
             <!--xacro:add_joint_names current_id="5" max_id="${link_qty}"/-->
         </plugin>
@@ -54,16 +46,3 @@
         <material>Gazebo/Blue</material>
     </gazebo>
-    <gazebo reference="link_2">
-        <material>Gazebo/Blue</material>
-    </gazebo>
-    <gazebo reference="link_3">
-        <material>Gazebo/Blue</material>
-    </gazebo>
-    <gazebo reference="link_4">
-        <material>Gazebo/Blue</material>
-    </gazebo>
-    <gazebo reference="link_5">
-        <material>Gazebo/Blue</material>
-    </gazebo>
-    <!--xacro:add_gazebo_links current_id="1" max_id="${link_qty}"/-->
 </robot>

File: description/robot.urdf.xacro (robot description, xacro)
@@ -153,7 +153,5 @@
 <xacro:property name="needle_radius" value="0.001" />
 <xacro:property name="needle_length" value="0.15" />
-<!-- Macro pour un maillon de l'aiguille -->
-<xacro:macro name="needle_link" params="id">
-    <link name="link_${id}">
+	<link name="link_1">
         <visual>
             <geometry>
@@ -161,8 +159,8 @@
             </geometry>
             <material name="blue"/>
-            <origin xyz="0 -0.075 0" rpy="0 1.5708 1.5708"/>
-        </visual>
-        <collision>
-            <origin xyz="0 -0.075 0" rpy="0 1.5708 1.5708"/>
+            <origin xyz="0 0 0" rpy="0 1.5708 1.5708"/>
+        </visual>
+        <collision>
+            <origin xyz="0 0 0" rpy="0 1.5708 1.5708"/>
             <geometry>
                 <box size="${link_y_size_x} ${link_y_size_y} ${link_y_size_z}"/>
@@ -170,47 +168,75 @@
         </collision>
         <xacro:inertial_cylinder mass="${needle_mass/link_qty}" length="${link_length}" radius="${link_radius}">
-            <origin xyz="0 -0.075 0" rpy="0 1.5708 1.5708"/>
+            <origin xyz="0 0 0" rpy="0 1.5708 1.5708"/>
         </xacro:inertial_cylinder>
     </link>
-    <!-- Joint to connect to the root link or previous link -->
-    <xacro:if value="${id == 1}">
-            <joint name="joint_needle" type="prismatic">
-            <parent link="link_y"/>
-            <child link="link_${id}"/>
-            <origin xyz="0 0 ${link_y_size_z/2}" rpy="0 0 0"/>
+    <joint name="joint_needle" type="prismatic">
+        <parent link="link_y"/>
+        <child link="link_1"/>
+        <origin xyz="0 0 ${link_y_size_z}" rpy="0 0 0"/>
+        <axis xyz="0 1 0"/>
+        <limit effort="1000" velocity="0.5" lower="-${needle_length}" upper="${needle_length/2}"/>
+    </joint>
+    <xacro:macro name="needle_link" params="base_name parent_name colour">
+        <link name="${base_name}_aux">
+            <visual>
+		        <geometry>
+		            <cylinder length="${link_length * 1/10}" radius="${link_radius}"/>
+		        </geometry>
+		        <origin xyz="0 0 0" rpy="0 1.5708 1.5708"/>
+		    </visual>
+		    <collision>
+		        <origin xyz="0 0 0" rpy="0 1.5708 1.5708"/>
+		        <geometry>
+		            <box size="${link_y_size_x} ${link_y_size_y} ${link_y_size_z}"/>
+		        </geometry>
+		    </collision>
+		    <xacro:inertial_cylinder mass="${needle_mass/link_qty}" length="${link_length}" radius="${link_radius}">
+		        <origin xyz="0 0 0" rpy="0 1.5708 1.5708"/>
+		    </xacro:inertial_cylinder>
+    	</link>
+    	<gazebo reference="${base_name}_aux">
+            <material>Gazebo/Black</material>
+            <self_collide>1</self_collide>
+        </gazebo>
+        <link name="${base_name}">
+     	    <visual>
+		        <geometry>
+		            <cylinder length="${link_length * 9/10}" radius="${link_radius}"/>
+		        </geometry>
+		        <origin xyz="0 0 0" rpy="0 1.5708 1.5708"/>
+		    </visual>
+		    <collision>
+		        <origin xyz="0 0 0" rpy="0 1.5708 1.5708"/>
+		        <geometry>
+		            <box size="${link_y_size_x} ${link_y_size_y} ${link_y_size_z}"/>
+		        </geometry>
+		    </collision>
+		    <xacro:inertial_cylinder mass="${needle_mass/link_qty}" length="${link_length}" radius="${link_radius}">
+		        <origin xyz="0 0 0" rpy="0 1.5708 1.5708"/>
+		    </xacro:inertial_cylinder>
+    	</link>
+    	<gazebo reference="${base_name}">
+            <material>Gazebo/${colour}</material>
+            <self_collide>1</self_collide>
+        </gazebo>
+        <joint name="${base_name}_aux_joint" type="revolute">
+            <parent link="${parent_name}"/>
+        	<child link="${base_name}_aux"/>
+            <origin xyz="0 ${link_length/2} 0" rpy="0 0 0"/>
+            <limit lower="-0.004" upper="0.004" effort="100.0" velocity="0.5"/>
+            <axis xyz="1 0 0"/>
+    	</joint>
+        <joint name="${base_name}_joint" type="revolute">
+    	    <parent link="${base_name}_aux"/>
+        	<child link="${base_name}"/>
+            <origin xyz="0 ${link_length/2} 0" rpy="0 0 0"/>
+            <limit lower="-0.004" upper="0.004" effort="100.0" velocity="0.5"/>
             <axis xyz="0 1 0"/>
-            <limit effort="1000" velocity="0.5" lower="-0.04" upper="${link_y_size_y}"/>
-        </joint>
-    </xacro:if>
-    <xacro:unless value="${id == 1}">
-        <xacro:universal_joint id="${id}"/>
-    </xacro:unless>
-</xacro:macro>
-<xacro:macro name="universal_joint" params="id">
-    <!-- Premier joint revolute autour de l'axe X -->
-    <joint name="joint_${id}_x" type="revolute">
-        <parent link="link_${id-1}"/>
-        <child link="link_${id}_x"/>
-        <origin xyz="0 ${link_length} 0" rpy="0 0 0"/>
-        <axis xyz="1 0 0"/>
-        <limit effort="30" velocity="0.5" lower="-1" upper="1"/>
-    </joint>
-    <link name="link_${id}_x">
-    </link>
-    <!-- Deuxième joint revolute autour de l'axe Z -->
-    <joint name="joint_${id}_z" type="revolute">
-        <parent link="link_${id}_x"/>
-        <child link="link_${id}"/>
-        <origin xyz="0 0 0" rpy="0 0 0"/>
-        <axis xyz="0 0 1"/>
-        <limit effort="30" velocity="0.5" lower="-1" upper="1"/>
-    </joint>
-</xacro:macro>
-<xacro:macro name="generate_links" params="current_link max_link">
-    <xacro:needle_link id="${current_link}"/>
-    <xacro:if value="${current_link != max_link}">
-        <xacro:generate_links current_link="${current_link + 1}" max_link="${max_link}"/>
-    </xacro:if>
-</xacro:macro>
-<xacro:generate_links current_link="1" max_link="${link_qty}"/>
+    	</joint>
+    </xacro:macro>
+    <xacro:needle_link base_name="link_2" parent_name="link_1" colour="Blue"/>
+    <xacro:needle_link base_name="link_3" parent_name="link_2" colour="Red"/>
+    <xacro:needle_link base_name="link_4" parent_name="link_3" colour="Purple"/>
+    <xacro:needle_link base_name="link_5" parent_name="link_4" colour="White"/>
 </robot>
