Commit message: Update gazebo_tags.xacro

File: description/gazebo_tags.xacro (robot description, xacro)
@@ -23,5 +23,13 @@
             <joint_name>joint_zx</joint_name>
             <joint_name>joint_needle</joint_name>
-            <xacro:add_joint_names current_id="2" max_id="${link_qty}"/>
+            <joint_name>joint_2_x</joint_name>
+            <joint_name>joint_3_x</joint_name>
+            <joint_name>joint_4_x</joint_name>
+            <joint_name>joint_5_x</joint_name>
+            <joint_name>joint_2_z</joint_name>
+            <joint_name>joint_3_z</joint_name>
+            <joint_name>joint_4_z</joint_name>
+            <joint_name>joint_5_z</joint_name>
+            <!--xacro:add_joint_names current_id="5" max_id="${link_qty}"/-->
         </plugin>
     </gazebo>
@@ -43,4 +51,19 @@
         <material>Gazebo/White</material>
     </gazebo>
-    <xacro:add_gazebo_links current_id="1" max_id="${link_qty}"/>
+    <gazebo reference="link_1">
+        <material>Gazebo/Blue</material>
+    </gazebo>
+    <gazebo reference="link_2">
+        <material>Gazebo/Blue</material>
+    </gazebo>
+    <gazebo reference="link_3">
+        <material>Gazebo/Blue</material>
+    </gazebo>
+    <gazebo reference="link_4">
+        <material>Gazebo/Blue</material>
+    </gazebo>
+    <gazebo reference="link_5">
+        <material>Gazebo/Blue</material>
+    </gazebo>
+    <!--xacro:add_gazebo_links current_id="1" max_id="${link_qty}"/-->
 </robot>

Commit message: No error, action server added, ready to use moveit . No real values, butr closer to the truth

File: description/gazebo_tags.xacro (robot description, xacro)
@@ -26,9 +26,4 @@
         </plugin>
     </gazebo>
-    <gazebo>
-        <plugin name="gazebo_ros_joint_pose_trajectory" filename="libgazebo_ros_joint_pose_trajectory.so">
-            <update_rate>20</update_rate>
-        </plugin>
-    </gazebo>
     <gazebo reference="base">
         <material>Gazebo/Orange</material>

File: description/robot.urdf.xacro (robot description, xacro)
@@ -3,5 +3,5 @@
     <xacro:include filename="inertial_macros.xacro"/>
     <xacro:include filename="gazebo_tags.xacro"/>
-    <xacro:include filename="gazebo_control.xacro"/>
+<!--  ***** ROBOT ASPECT  *****   -->
     <!-- colors-->
     <material name="white">
@@ -14,5 +14,5 @@
         <color rgba="0.2 0.2 1 1"/>
     </material>
-    <!-- measures-->
+    <!-- measures -->
     <xacro:property name="base_size_x_half" value="0.0655" />
     <xacro:property name="base_size_y_half" value="0.1905" />
@@ -29,10 +29,17 @@
     <xacro:property name="x_offset" value="0.007" />
     <xacro:property name="y_offset" value="0.006" />
-    <xacro:property name="mass_base" value="0.4" />
+    <xacro:property name="mass_base" value="0.04" />
     <xacro:property name="mass_x" value="0.3" />
     <xacro:property name="mass_y" value="0.3" />
     <xacro:property name="mass_z" value="0.25" />
+    <!-- measures for the needle -->
     <xacro:property name="needle_mass" value="0.006" />
-    <!-- links and bases-->
+    <xacro:property name="link_qty" value="5"/>
+	<xacro:property name="link_length" value="${needle_length/ link_qty}"/>
+	<xacro:property name="link_radius" value="${needle_radius}"/>
+	<xacro:property name="link_mass" value="needle_mass/link_qty"/>
+	<xacro:property name="needle_radius" value="0.001" />
+	<xacro:property name="needle_length" value="0.15" />
+    <!-- links and bases -->
     <link name="dummy_link"/>
     <joint name="dummy_joint" type="fixed">
@@ -86,5 +93,5 @@
         <child link="link_x" />
         <axis xyz="0 0 1" />
-        <limit effort="100" lower="-${base_size_z/2 + link_z_size_z/2 - link_x_size_z}" upper="${base_size_z/2 + link_z_size_z/2 - link_x_size_z}" velocity="100"  />
+        <limit effort="100" lower="-${base_size_z/2 + link_z_size_z/2 - link_x_size_z}" upper="${base_size_z/2 + link_z_size_z/2 - link_x_size_z}" velocity="0.1"  />
     </joint>
     <link name="link_x">
@@ -111,5 +118,5 @@
         <origin xyz="-${link_z_size_x/2 + link_x_size_x/2}  0 0" rpy="0 0 0" />
         <axis xyz="1 0 0" />
-        <limit effort="1000.0" lower="-${link_z_size_x/2 + link_x_size_x/2 - link_z_size_x/2}" upper="${link_z_size_x/2 + link_x_size_x/2 - link_z_size_x/2}" velocity="0.5"  />
+        <limit effort="1000.0" lower="-${link_z_size_x/2 + link_x_size_x/2 - link_z_size_x/2}" upper="${link_z_size_x/2 + link_x_size_x/2 - link_z_size_x/2}" velocity="0.1"  />
     </joint>
     <link name="link_y">
@@ -136,5 +143,5 @@
         <origin xyz="0 0 ${link_y_size_z/2}" rpy="0 0 0" />
         <axis xyz="0 1 0" />
-        <limit effort="1000.0" lower="0.045" upper="0.12" velocity="0.5"  />
+        <limit effort="1000.0" lower="0.045" upper="0.12" velocity="0.1"  />
     </joint>
     <link name="needle">
@@ -147,10 +154,5 @@
         </visual>
     </link-->
-<xacro:property name="link_qty" value="5"/>
-<xacro:property name="link_length" value="${needle_length/ link_qty}"/>
-<xacro:property name="link_radius" value="${needle_radius}"/>
-<xacro:property name="link_mass" value="needle_mass/link_qty"/>
-<xacro:property name="needle_radius" value="0.001" />
-<xacro:property name="needle_length" value="0.15" />
+	<!-- constuction of the articulated needle -->
 	<link name="link_1">
         <visual>
@@ -158,5 +160,4 @@
                 <cylinder length="${link_length}" radius="${link_radius}"/>
             </geometry>
-            <material name="blue"/>
             <origin xyz="0 0 0" rpy="0 1.5708 1.5708"/>
         </visual>
@@ -176,25 +177,37 @@
         <origin xyz="0 0 ${link_y_size_z}" rpy="0 0 0"/>
         <axis xyz="0 1 0"/>
-        <limit effort="1000" velocity="0.5" lower="-${needle_length}" upper="${needle_length/2}"/>
-    </joint>
+        <limit effort="1000" velocity="0.1" lower="-${needle_length}" upper="${needle_length/2}"/>
+    </joint>
+    <gazebo reference="link_1">
+        <kp>1.0</kp>
+        <kd>1.0</kd>
+        <mu1>1000.0</mu1>
+        <mu2>1000.0</mu2>
+        <material>Gazebo/Green</material>
+        <self_collide>1</self_collide>
+    </gazebo>
     <xacro:macro name="needle_link" params="base_name parent_name colour">
         <link name="${base_name}_aux">
             <visual>
-		        <geometry>
-		            <cylinder length="${link_length * 1/10}" radius="${link_radius}"/>
-		        </geometry>
-		        <origin xyz="0 0 0" rpy="0 1.5708 1.5708"/>
-		    </visual>
-		    <collision>
-		        <origin xyz="0 0 0" rpy="0 1.5708 1.5708"/>
-		        <geometry>
-		            <box size="${link_y_size_x} ${link_y_size_y} ${link_y_size_z}"/>
-		        </geometry>
-		    </collision>
-		    <xacro:inertial_cylinder mass="${needle_mass/link_qty}" length="${link_length}" radius="${link_radius}">
-		        <origin xyz="0 0 0" rpy="0 1.5708 1.5708"/>
-		    </xacro:inertial_cylinder>
-    	</link>
+	        <geometry>
+	            <cylinder length="${link_length * 1/10}" radius="${link_radius}"/>
+	        </geometry>
+	        <origin xyz="0 0 0" rpy="0 1.5708 1.5708"/>
+	    </visual>
+	    <collision>
+	        <origin xyz="0 0 0" rpy="0 1.5708 1.5708"/>
+	        <geometry>
+	            <box size="${link_y_size_x} ${link_y_size_y} ${link_y_size_z}"/>
+	        </geometry>
+	    </collision>
+	    <xacro:inertial_cylinder mass="${needle_mass/link_qty}" length="${link_length}" radius="${link_radius}">
+	        <origin xyz="0 0 0" rpy="0 1.5708 1.5708"/>
+	    </xacro:inertial_cylinder>
+	</link>
     	<gazebo reference="${base_name}_aux">
+    		<kp>1.0</kp>
+            <kd>1.0</kd>
+            <mu1>1000.0</mu1>
+            <mu2>1000.0</mu2>
             <material>Gazebo/Black</material>
             <self_collide>1</self_collide>
@@ -202,20 +215,24 @@
         <link name="${base_name}">
      	    <visual>
-		        <geometry>
-		            <cylinder length="${link_length * 9/10}" radius="${link_radius}"/>
-		        </geometry>
-		        <origin xyz="0 0 0" rpy="0 1.5708 1.5708"/>
-		    </visual>
-		    <collision>
-		        <origin xyz="0 0 0" rpy="0 1.5708 1.5708"/>
-		        <geometry>
-		            <box size="${link_y_size_x} ${link_y_size_y} ${link_y_size_z}"/>
-		        </geometry>
-		    </collision>
-		    <xacro:inertial_cylinder mass="${needle_mass/link_qty}" length="${link_length}" radius="${link_radius}">
-		        <origin xyz="0 0 0" rpy="0 1.5708 1.5708"/>
-		    </xacro:inertial_cylinder>
+	        <geometry>
+	            <cylinder length="${link_length * 9/10}" radius="${link_radius}"/>
+	        </geometry>
+	        <origin xyz="0 0 0" rpy="0 1.5708 1.5708"/>
+	    </visual>
+	    <collision>
+	        <origin xyz="0 0 0" rpy="0 1.5708 1.5708"/>
+	        <geometry>
+	            <box size="${link_y_size_x} ${link_y_size_y} ${link_y_size_z}"/>
+	        </geometry>
+	    </collision>
+	    <xacro:inertial_cylinder mass="${needle_mass/link_qty}" length="${link_length}" radius="${link_radius}">
+	        <origin xyz="0 0 0" rpy="0 1.5708 1.5708"/>
+	    </xacro:inertial_cylinder>
     	</link>
     	<gazebo reference="${base_name}">
+    		<kp>1.0</kp>
+            <kd>1.0</kd>
+            <mu1>1000.0</mu1>
+            <mu2>1000.0</mu2>
             <material>Gazebo/${colour}</material>
             <self_collide>1</self_collide>
@@ -225,5 +242,5 @@
         	<child link="${base_name}_aux"/>
             <origin xyz="0 ${link_length/2} 0" rpy="0 0 0"/>
-            <limit lower="-0.004" upper="0.004" effort="100.0" velocity="0.5"/>
+            <limit lower="-0.04" upper="0.04" effort="100.0" velocity="0.1"/>
             <axis xyz="1 0 0"/>
     	</joint>
@@ -232,11 +249,131 @@
         	<child link="${base_name}"/>
             <origin xyz="0 ${link_length/2} 0" rpy="0 0 0"/>
-            <limit lower="-0.004" upper="0.004" effort="100.0" velocity="0.5"/>
+            <limit lower="-0.04" upper="0.04" effort="100.0" velocity="0.1"/>
             <axis xyz="0 1 0"/>
     	</joint>
+    	<transmission name="tran${base_name}_aux">
+            <type>transmission_interface/SimpleTransmission</type>
+            <joint name="${base_name}_aux_joint">
+                <hardwareInterface>EffortJointInterface</hardwareInterface>
+            </joint>
+            <actuator name="motor${base_name}_aux">
+                <hardwareInterface>EffortJointInterface</hardwareInterface>
+                <mechanicalReduction>1</mechanicalReduction>
+            </actuator>
+        </transmission>
+        <transmission name="tran${base_name}">
+            <type>transmission_interface/SimpleTransmission</type>
+            <joint name="${base_name}_joint">
+                <hardwareInterface>EffortJointInterface</hardwareInterface>
+            </joint>
+            <actuator name="motor${base_name}">
+                <hardwareInterface>EffortJointInterface</hardwareInterface>
+                <mechanicalReduction>1</mechanicalReduction>
+            </actuator>
+        </transmission>
     </xacro:macro>
+    <!-- initialisation of the needle-->
     <xacro:needle_link base_name="link_2" parent_name="link_1" colour="Blue"/>
     <xacro:needle_link base_name="link_3" parent_name="link_2" colour="Red"/>
     <xacro:needle_link base_name="link_4" parent_name="link_3" colour="Purple"/>
     <xacro:needle_link base_name="link_5" parent_name="link_4" colour="White"/>
+<!--  ***** ROS2 GAZEBO CONTROL PACKAGE  *****   -->
+    <ros2_control name="GazeboSystem" type="system">
+        <hardware>
+            <plugin>gazebo_ros2_control/GazeboSystem</plugin>
+        </hardware>
+        <joint name="joint_zx">
+            <command_interface name="position">
+                <param name="min">-${base_size_z/2 + link_z_size_z/2 - link_x_size_z}"</param>
+                <param name="max">"${base_size_z/2 + link_z_size_z/2 - link_x_size_z}"</param>
+            </command_interface>
+            <state_interface name="position"/>
+            <state_interface name="velocity"/>
+        </joint>
+        <joint name="joint_xy">
+            <command_interface name="position">
+                <param name="min">-${link_z_size_x/2 + link_x_size_x/2 - link_z_size_x/2}</param>
+                <param name="max">${link_z_size_x/2 + link_x_size_x/2 - link_z_size_x/2}</param>
+            </command_interface>
+            <state_interface name="position"/> <!--what I want to broadcast-->
+            <state_interface name="velocity"/>
+        </joint>
+        <joint name="joint_needle">
+            <command_interface name="position">
+                <param name="min">-${needle_length}</param>
+                <param name="max">${needle_length/2}</param>
+            </command_interface>
+            <state_interface name="position"/>
+            <state_interface name="velocity"/>
+        </joint>
+        <joint name="link_2_aux_joint">
+            <command_interface name="position">
+                <param name="min">-0.04</param>
+                <param name="max">0.04</param>
+            </command_interface>
+            <state_interface name="position"/>
+            <state_interface name="velocity"/>
+        </joint>
+        <joint name="link_2_joint">
+            <command_interface name="position">
+                <param name="min">-0.04</param>
+                <param name="max">0.04</param>
+            </command_interface>
+            <state_interface name="position"/>
+            <state_interface name="velocity"/>
+        </joint>
+        <joint name="link_3_aux_joint">
+            <command_interface name="position">
+                <param name="min">-0.04</param>
+                <param name="max">0.04</param>
+            </command_interface>
+            <state_interface name="position"/>
+            <state_interface name="velocity"/>
+        </joint>
+        <joint name="link_3_joint">
+            <command_interface name="position">
+                <param name="min">-0.04</param>
+                <param name="max">0.04</param>
+            </command_interface>
+            <state_interface name="position"/>
+            <state_interface name="velocity"/>
+        </joint>
+        <joint name="link_4_aux_joint">
+            <command_interface name="position">
+                <param name="min">-0.04</param>
+                <param name="max">0.04</param>
+            </command_interface>
+            <state_interface name="position"/>
+            <state_interface name="velocity"/>
+        </joint>
+        <joint name="link_4_joint">
+            <command_interface name="position">
+                <param name="min">-0.04</param>
+                <param name="max">0.04</param>
+            </command_interface>
+            <state_interface name="position"/>
+            <state_interface name="velocity"/>
+        </joint>
+        <joint name="link_5_aux_joint">
+            <command_interface name="position">
+                <param name="min">-0.04</param>
+                <param name="max">0.04</param>
+            </command_interface>
+            <state_interface name="position"/>
+            <state_interface name="velocity"/>
+        </joint>
+        <joint name="link_5_joint">
+            <command_interface name="position">
+                <param name="min">-0.04</param>
+                <param name="max">0.04</param>
+            </command_interface>
+            <state_interface name="position"/>
+            <state_interface name="velocity"/>
+        </joint>
+    </ros2_control>
+    <gazebo>
+        <plugin filename="libgazebo_ros2_control.so" name="gazebo_ros2_control">
+            <parameters>$(find my_bot)/config/controller.yaml</parameters>
+        </plugin>
+    </gazebo>
 </robot>
