Commit message: Update robot.urdf.xacro

File: description/robot.urdf.xacro (robot description, xacro)
@@ -1,2 +1,106 @@
+<?xml version="1.0"?>
+<robot xmlns:xacro="http://www.ros.org/wiki/xacro" name="robot">
+    <!-- colors-->
+    <material name="white">
+        <color rgba="1 1 1 1"/>
+    </material>
+    <material name="orange">
+        <color rgba="1 0.3 0.1 1"/>
+    </material>
+    <material name="blue">
+        <color rgba="0.2 0.2 1 1"/>
+    </material>
+    <!-- mesures-->
+    <xacro:property name="base_size_x_half" value="0.0655" />
+    <xacro:property name="base_size_y_half" value="0.1905" />
+    <xacro:property name="base_size_z" value="0.026" />
+    <xacro:property name="link_z_size_x" value="0.019" />
+    <xacro:property name="link_z_size_y" value="0.038" />
+    <xacro:property name="link_z_size_z" value="0.14" />
+    <xacro:property name="link_x_size_x" value="0.092" />
+    <xacro:property name="link_x_size_y" value="0.038" />
+    <xacro:property name="link_x_size_z" value="0.025" />
+    <xacro:property name="link_y_size_x" value="0.045" />
+    <xacro:property name="link_y_size_y" value="0.3" />
+    <xacro:property name="link_y_size_z" value="0.01" />
+    <xacro:property name="x_offset" value="0.007" />
+    <xacro:property name="y_offset" value="0.006" />
+    <!-- links and bases-->
+    <link name="base">
+        <visual>
+            <geometry>
+                <box size="${base_size_x_half * 2} ${base_size_y_half * 2} ${base_size_z}" />
+            </geometry>
+            <material name="orange" />
+        </visual>
+    </link>
+    <joint name="base_joint" type="fixed">
+        <parent link="base" />
+        <child link="link_z" />
+        <origin xyz="${base_size_x_half - link_z_size_x/2 - x_offset} -${base_size_y_half - link_z_size_y/2 - y_offset} 0.0" />
+    </joint>
+    <link name="link_z">
+        <visual>
+            <origin xyz="0 0 ${base_size_z/2 + link_z_size_z/2}" rpy="0.0 0.0 0.0"  />
+            <geometry>
+                <box size="${link_z_size_x} ${link_z_size_y} ${link_z_size_z}" />
+            </geometry>
+            <material name="white"/>
+        </visual>
+    </link>
+    <joint name="joint_zx" type="prismatic">
+        <origin xyz="0 0 ${base_size_z/2 + link_z_size_z/2}" />
+        <parent link="link_z" />
+        <child link="link_x" />
+        <axis xyz="0 0 1" />
+        <limit effort="100" lower="-${base_size_z/2 + link_z_size_z/2 - link_x_size_z}" upper="${base_size_z/2 + link_z_size_z/2 - link_x_size_z}" velocity="100"  />
+    </joint>
+    <link name="link_x">
+        <visual>
+            <origin xyz="-${link_z_size_x/2 + link_x_size_x/2} 0 0" rpy="0 0 0"  />
+            <geometry>
+                <box size="${link_x_size_x} ${link_x_size_y} ${link_x_size_z}" />
+            </geometry>
+            <material name="white"/>
+        </visual>
+    </link>
+    <joint name="joint_xy" type="prismatic">
+        <parent link="link_x" />
+        <child link="link_y" />
+        <origin xyz="-${link_z_size_x/2 + link_x_size_x/2}  0 0" rpy="0 0 0" />
+        <axis xyz="1 0 0" />
+        <limit effort="1000.0" lower="-${link_z_size_x/2 + link_x_size_x/2 - link_z_size_x/2}" upper="${link_z_size_x/2 + link_x_size_x/2 - link_z_size_x/2}" velocity="0.5"  />
+    </joint>
+    <link name="link_y">
+        <visual>
+            <origin xyz="0 ${link_y_size_y/2 + link_x_size_y/2}  0" />
+            <geometry>
+                <box size="${link_y_size_x} ${link_y_size_y} ${link_y_size_z}"  />
+            </geometry>
+            <material name="white"/>
+        </visual>
+    </link>
+    <!--joint name="joint_y" type="prismatic">
+        <parent link="link_y" />
+        <child link="needle" />
+        <origin xyz="0 0 ${link_y_size_z/2}" rpy="0 0 0" />
+        <axis xyz="0 1 0" />
+        <limit effort="1000.0" lower="0.045" upper="0.12" velocity="0.5"  />
+    </joint>
+    <link name="needle">
+        <visual>
+            <origin xyz="0 -0.075 0" rpy="1.5708 0 0"/>
+            <geometry>
+                <cylinder radius="${needle_radius}" length = "${needle_length}" />
+            </geometry>
+            <material name="blue"/>
+        </visual>
+    </link-->
+<xacro:property name="link_qty" value="2"/>
+<xacro:property name="link_length" value="${needle_length/ link_qty}"/>
+<xacro:property name="link_radius" value="${needle_radius}"/>
+<xacro:property name="link_mass" value="0.01"/>
+<xacro:property name="needle_radius" value="0.001" />
+<xacro:property name="needle_length" value="0.15" />
 <!-- Macro pour un maillon du serpent -->
 <xacro:macro name="needle_link" params="id">
@@ -10,7 +114,7 @@
         </visual>
     </link>
-    <!-- Joint pour se connecter au maillon racine ou précédent -->
+    <!-- Joint to connect to the root link or previous link -->
     <xacro:if value="${id == 1}">
-        <joint name="joint_needle" type="prismatic">
+            <joint name="joint_needle" type="prismatic">
             <parent link="link_y"/>
             <child link="link_${id}"/>
@@ -21,27 +125,12 @@
     </xacro:if>
     <xacro:unless value="${id == 1}">
-        <xacro:universal_joint id="${id}"/>
+        <joint name="joint_${id-1}_${id}" type="revolute">
+            <parent link="link_${id-1}"/>
+            <child link="link_${id}"/>
+            <origin xyz="0 ${link_length} 0" rpy="0 0 0"/>
+            <axis xyz="0 0 1"/>
+            <limit effort="30" velocity="0.5" lower="-${needle_radius * 70}" upper="${needle_radius * 70}"/>
+        </joint>
     </xacro:unless>
-</xacro:macro>
-<xacro:macro name="universal_joint" params="id">
-    <!-- Premier joint revolute autour de l'axe X -->
-    <joint name="joint_${id}_x" type="revolute">
-        <parent link="link_${id-1}"/>
-        <child link="link_${id}_x"/>
-        <origin xyz="0 ${link_length} 0" rpy="0 0 0"/>
-        <axis xyz="1 0 0"/>
-        <limit effort="30" velocity="0.5"/>
-    </joint>
-    <link name="link_${id}_x">
-        <!-- vous pouvez ajouter des visuels si nécessaire -->
-    </link>
-    <!-- Deuxième joint revolute autour de l'axe Z -->
-    <joint name="joint_${id}_z" type="revolute">
-        <parent link="link_${id}_x"/>
-        <child link="link_${id}"/>
-        <origin xyz="0 0 0" rpy="0 0 0"/>
-        <axis xyz="0 0 1"/>
-        <limit effort="30" velocity="0.5"/>
-    </joint>
 </xacro:macro>
 <xacro:macro name="generate_links" params="current_link max_link">
@@ -52,2 +141,3 @@
 </xacro:macro>
 <xacro:generate_links current_link="1" max_link="${link_qty}"/>
+</robot>

Commit message: Update robot.urdf.xacro

File: description/robot.urdf.xacro (robot description, xacro)
@@ -1,8 +1,224 @@
 <?xml version="1.0"?>
 <robot xmlns:xacro="http://www.ros.org/wiki/xacro" name="robot">
+<<<<<<< HEAD
+    <xacro:include filename="inertial_macros.xacro"/>
+    <xacro:include filename="gazebo_tags.xacro"/>
+    <xacro:include filename="gazebo_control.xacro"/>
     <!-- colors-->
     <material name="white">
         <color rgba="1 1 1 1"/>
     </material>
+    <material name="orange">
+        <color rgba="1 0.3 0.1 1"/>
+    </material>
+    <material name="blue">
+        <color rgba="0.2 0.2 1 1"/>
+    </material>
+    <!-- measures-->
+    <xacro:property name="base_size_x_half" value="0.0655" />
+    <xacro:property name="base_size_y_half" value="0.1905" />
+    <xacro:property name="base_size_z" value="0.026" />
+    <xacro:property name="link_z_size_x" value="0.019" />
+    <xacro:property name="link_z_size_y" value="0.038" />
+    <xacro:property name="link_z_size_z" value="0.14" />
+    <xacro:property name="link_x_size_x" value="0.092" />
+    <xacro:property name="link_x_size_y" value="0.038" />
+    <xacro:property name="link_x_size_z" value="0.025" />
+    <xacro:property name="link_y_size_x" value="0.045" />
+    <xacro:property name="link_y_size_y" value="0.3" />
+    <xacro:property name="link_y_size_z" value="0.01" />
+    <xacro:property name="x_offset" value="0.007" />
+    <xacro:property name="y_offset" value="0.006" />
+    <xacro:property name="mass_base" value="0.2" />
+    <xacro:property name="mass_x" value="0.1" />
+    <xacro:property name="mass_y" value="0.1" />
+    <xacro:property name="mass_z" value="0.15" />
+    <xacro:property name="needle_mass" value="0.006" />
+    <!-- links and bases-->
+    <link name="dummy_link"/>
+    <joint name="dummy_joint" type="fixed">
+        <parent link="dummy_link"/>
+        <child link="base"/>
+        <origin xyz="0 0 0" rpy="0 0 0"/>
+    </joint>
+    <link name="base">
+        <visual>
+            <geometry>
+                <box size="${base_size_x_half * 2} ${base_size_y_half * 2} ${base_size_z}" />
+            </geometry>
+            <material name="orange" />
+        </visual>
+        <collision>
+            <origin xyz="0 0 0" rpy="0 0 0"/>
+            <geometry>
+                <box size="${base_size_x_half * 2} ${base_size_y_half * 2} ${base_size_z}"/>
+            </geometry>
+        </collision>
+        <xacro:inertial_box mass="${mass_base}" x="${base_size_x_half * 2}" y="${base_size_y_half * 2}" z="${base_size_z * 2}">
+            <origin xyz="0 0 0" rpy="0 0 0"/>
+        </xacro:inertial_box>
+    </link>
+    <joint name="base_joint" type="fixed">
+        <parent link="base" />
+        <child link="link_z" />
+        <origin xyz="${base_size_x_half - link_z_size_x/2 - x_offset} -${base_size_y_half - link_z_size_y/2 - y_offset} 0.0" />
+    </joint>
+    <link name="link_z">
+        <visual>
+            <origin xyz="0 0 ${base_size_z/2 + link_z_size_z/2}" rpy="0.0 0.0 0.0"  />
+            <geometry>
+                <box size="${link_z_size_x} ${link_z_size_y} ${link_z_size_z}" />
+            </geometry>
+            <material name="white"/>
+        </visual>
+        <collision>
+            <origin xyz="0 0 ${base_size_z/2 + link_z_size_z/2}" rpy="0 0 0"/>
+            <geometry>
+                <box size="${link_z_size_x} ${link_z_size_y} ${link_z_size_z}"/>
+            </geometry>
+        </collision>
+        <xacro:inertial_box mass="${mass_z}" x="${link_z_size_x}" y="${link_z_size_y}" z="${link_z_size_z}">
+            <origin xyz="0 0 ${base_size_z/2 + link_z_size_z/2}" rpy="0 0 0"/>
+        </xacro:inertial_box>
+    </link>
+    <joint name="joint_zx" type="prismatic">
+        <origin xyz="0 0 ${base_size_z/2 + link_z_size_z/2}" />
+        <parent link="link_z" />
+        <child link="link_x" />
+        <axis xyz="0 0 1" />
+        <limit effort="100" lower="-${base_size_z/2 + link_z_size_z/2 - link_x_size_z}" upper="${base_size_z/2 + link_z_size_z/2 - link_x_size_z}" velocity="100"  />
+    </joint>
+    <link name="link_x">
+        <visual>
+            <origin xyz="-${link_z_size_x/2 + link_x_size_x/2} 0 0" rpy="0 0 0"  />
+            <geometry>
+                <box size="${link_x_size_x} ${link_x_size_y} ${link_x_size_z}" />
+            </geometry>
+            <material name="white"/>
+        </visual>
+        <collision>
+            <origin xyz="-${link_z_size_x/2 + link_x_size_x/2} 0 0" rpy="0 0 0"/>
+            <geometry>
+                <box size="${link_x_size_x} ${link_x_size_y} ${link_x_size_z}"/>
+            </geometry>
+        </collision>
+        <xacro:inertial_box mass="${mass_x}" x="${link_x_size_x}" y="${link_x_size_y}" z="${link_x_size_z}">
+            <origin xyz="-${link_z_size_x/2 + link_x_size_x/2} 0 0" rpy="0 0 0"/>
+        </xacro:inertial_box>
+    </link>
+    <joint name="joint_xy" type="prismatic">
+        <parent link="link_x" />
+        <child link="link_y" />
+        <origin xyz="-${link_z_size_x/2 + link_x_size_x/2}  0 0" rpy="0 0 0" />
+        <axis xyz="1 0 0" />
+        <limit effort="1000.0" lower="-${link_z_size_x/2 + link_x_size_x/2 - link_z_size_x/2}" upper="${link_z_size_x/2 + link_x_size_x/2 - link_z_size_x/2}" velocity="0.5"  />
+    </joint>
+    <link name="link_y">
+        <visual>
+            <origin xyz="0 ${link_y_size_y/2 + link_x_size_y/2}  0" />
+            <geometry>
+                <box size="${link_y_size_x} ${link_y_size_y} ${link_y_size_z}"  />
+            </geometry>
+            <material name="white"/>
+        </visual>
+        <collision>
+            <origin xyz="0 ${link_y_size_y/2 + link_x_size_y/2}  0" rpy="0 0 0"/>
+            <geometry>
+                <box size="${link_y_size_x} ${link_y_size_y} ${link_y_size_z}"/>
+            </geometry>
+        </collision>
+        <xacro:inertial_box mass="${mass_y}" x="${link_y_size_x}" y="${link_y_size_y}" z="${link_y_size_z}">
+            <origin xyz="0 ${link_y_size_y/2 + link_x_size_y/2}  0" rpy="0 0 0"/>
+        </xacro:inertial_box>
+    </link>
+    <!--joint name="joint_y" type="prismatic">
+        <parent link="link_y" />
+        <child link="needle" />
+        <origin xyz="0 0 ${link_y_size_z/2}" rpy="0 0 0" />
+        <axis xyz="0 1 0" />
+        <limit effort="1000.0" lower="0.045" upper="0.12" velocity="0.5"  />
+    </joint>
+    <link name="needle">
+        <visual>
+            <origin xyz="0 -0.075 0" rpy="1.5708 0 0"/>
+            <geometry>
+                <cylinder radius="${needle_radius}" length = "${needle_length}" />
+            </geometry>
+            <material name="blue"/>
+        </visual>
+    </link-->
+<xacro:property name="link_qty" value="5"/>
+<xacro:property name="link_length" value="${needle_length/ link_qty}"/>
+<xacro:property name="link_radius" value="${needle_radius}"/>
+<xacro:property name="link_mass" value="0.01"/>
+<xacro:property name="needle_radius" value="0.001" />
+<xacro:property name="needle_length" value="0.15" />
+<!-- Macro pour un maillon de l'aiguille -->
+<xacro:macro name="needle_link" params="id">
+    <link name="link_${id}">
+        <visual>
+            <geometry>
+                <cylinder length="${link_length}" radius="${link_radius}"/>
+            </geometry>
+            <material name="blue"/>
+            <origin xyz="0 -0.075 0" rpy="0 1.5708 1.5708"/>
+        </visual>
+        <collision>
+            <origin xyz="0 -0.075 0" rpy="0 1.5708 1.5708"/>
+            <geometry>
+                <box size="${link_y_size_x} ${link_y_size_y} ${link_y_size_z}"/>
+            </geometry>
+        </collision>
+        <xacro:inertial_cylinder mass="${needle_mass/link_qty}" length="${link_length}" radius="${link_radius}">
+            <origin xyz="0 -0.075 0" rpy="0 1.5708 1.5708"/>
+        </xacro:inertial_cylinder>
+    </link>
+    <!-- Joint to connect to the root link or previous link -->
+    <xacro:if value="${id == 1}">
+            <joint name="joint_needle" type="prismatic">
+            <parent link="link_y"/>
+            <child link="link_${id}"/>
+            <origin xyz="0 0 ${link_y_size_z/2}" rpy="0 0 0"/>
+            <axis xyz="0 1 0"/>
+            <limit effort="1000" velocity="0.5" lower="-0.04" upper="${link_y_size_y}"/>
+        </joint>
+    </xacro:if>
+    <xacro:unless value="${id == 1}">
+        <xacro:universal_joint id="${id}"/>
+    </xacro:unless>
+</xacro:macro>
+<xacro:macro name="universal_joint" params="id">
+    <!-- Premier joint revolute autour de l'axe X -->
+    <joint name="joint_${id}_x" type="revolute">
+        <parent link="link_${id-1}"/>
+        <child link="link_${id}_x"/>
+        <origin xyz="0 ${link_length} 0" rpy="0 0 0"/>
+        <axis xyz="1 0 0"/>
+        <limit effort="30" velocity="0.5" lower="-1" upper="1"/>
+    </joint>
+    <link name="link_${id}_x">
+    </link>
+    <!-- Deuxième joint revolute autour de l'axe Z -->
+    <joint name="joint_${id}_z" type="revolute">
+        <parent link="link_${id}_x"/>
+        <child link="link_${id}"/>
+        <origin xyz="0 0 0" rpy="0 0 0"/>
+        <axis xyz="0 0 1"/>
+        <limit effort="30" velocity="0.5" lower="-1" upper="1"/>
+    </joint>
+</xacro:macro>
+<xacro:macro name="generate_links" params="current_link max_link">
+    <xacro:needle_link id="${current_link}"/>
+    <xacro:if value="${current_link != max_link}">
+        <xacro:generate_links current_link="${current_link + 1}" max_link="${max_link}"/>
+    </xacro:if>
+</xacro:macro>
+<xacro:generate_links current_link="1" max_link="${link_qty}"/>
+=======
+    <!-- colors-->
+    <material name="white">
+        <color rgba="1 1 1 1"/>
+    </material>
+>>>>>>> 0d3edb151c2043f0e1971c84f5d1e92f0bc8fb51
     <material name="orange">
         <color rgba="1 0.3 0.1 1"/>

Commit message: Update robot.urdf.xacro

File: description/robot.urdf.xacro (robot description, xacro)
@@ -215,145 +215,3 @@
 </xacro:macro>
 <xacro:generate_links current_link="1" max_link="${link_qty}"/>
-=======
-    <!-- colors-->
-    <material name="white">
-        <color rgba="1 1 1 1"/>
-    </material>
->>>>>>> 0d3edb151c2043f0e1971c84f5d1e92f0bc8fb51
-    <material name="orange">
-        <color rgba="1 0.3 0.1 1"/>
-    </material>
-    <material name="blue">
-        <color rgba="0.2 0.2 1 1"/>
-    </material>
-    <!-- mesures-->
-    <xacro:property name="base_size_x_half" value="0.0655" />
-    <xacro:property name="base_size_y_half" value="0.1905" />
-    <xacro:property name="base_size_z" value="0.026" />
-    <xacro:property name="link_z_size_x" value="0.019" />
-    <xacro:property name="link_z_size_y" value="0.038" />
-    <xacro:property name="link_z_size_z" value="0.14" />
-    <xacro:property name="link_x_size_x" value="0.092" />
-    <xacro:property name="link_x_size_y" value="0.038" />
-    <xacro:property name="link_x_size_z" value="0.025" />
-    <xacro:property name="link_y_size_x" value="0.045" />
-    <xacro:property name="link_y_size_y" value="0.3" />
-    <xacro:property name="link_y_size_z" value="0.01" />
-    <xacro:property name="x_offset" value="0.007" />
-    <xacro:property name="y_offset" value="0.006" />
-    <!-- links and bases-->
-    <link name="base">
-        <visual>
-            <geometry>
-                <box size="${base_size_x_half * 2} ${base_size_y_half * 2} ${base_size_z}" />
-            </geometry>
-            <material name="orange" />
-        </visual>
-    </link>
-    <joint name="base_joint" type="fixed">
-        <parent link="base" />
-        <child link="link_z" />
-        <origin xyz="${base_size_x_half - link_z_size_x/2 - x_offset} -${base_size_y_half - link_z_size_y/2 - y_offset} 0.0" />
-    </joint>
-    <link name="link_z">
-        <visual>
-            <origin xyz="0 0 ${base_size_z/2 + link_z_size_z/2}" rpy="0.0 0.0 0.0"  />
-            <geometry>
-                <box size="${link_z_size_x} ${link_z_size_y} ${link_z_size_z}" />
-            </geometry>
-            <material name="white"/>
-        </visual>
-    </link>
-    <joint name="joint_zx" type="prismatic">
-        <origin xyz="0 0 ${base_size_z/2 + link_z_size_z/2}" />
-        <parent link="link_z" />
-        <child link="link_x" />
-        <axis xyz="0 0 1" />
-        <limit effort="100" lower="-${base_size_z/2 + link_z_size_z/2 - link_x_size_z}" upper="${base_size_z/2 + link_z_size_z/2 - link_x_size_z}" velocity="100"  />
-    </joint>
-    <link name="link_x">
-        <visual>
-            <origin xyz="-${link_z_size_x/2 + link_x_size_x/2} 0 0" rpy="0 0 0"  />
-            <geometry>
-                <box size="${link_x_size_x} ${link_x_size_y} ${link_x_size_z}" />
-            </geometry>
-            <material name="white"/>
-        </visual>
-    </link>
-    <joint name="joint_xy" type="prismatic">
-        <parent link="link_x" />
-        <child link="link_y" />
-        <origin xyz="-${link_z_size_x/2 + link_x_size_x/2}  0 0" rpy="0 0 0" />
-        <axis xyz="1 0 0" />
-        <limit effort="1000.0" lower="-${link_z_size_x/2 + link_x_size_x/2 - link_z_size_x/2}" upper="${link_z_size_x/2 + link_x_size_x/2 - link_z_size_x/2}" velocity="0.5"  />
-    </joint>
-    <link name="link_y">
-        <visual>
-            <origin xyz="0 ${link_y_size_y/2 + link_x_size_y/2}  0" />
-            <geometry>
-                <box size="${link_y_size_x} ${link_y_size_y} ${link_y_size_z}"  />
-            </geometry>
-            <material name="white"/>
-        </visual>
-    </link>
-    <!--joint name="joint_y" type="prismatic">
-        <parent link="link_y" />
-        <child link="needle" />
-        <origin xyz="0 0 ${link_y_size_z/2}" rpy="0 0 0" />
-        <axis xyz="0 1 0" />
-        <limit effort="1000.0" lower="0.045" upper="0.12" velocity="0.5"  />
-    </joint>
-    <link name="needle">
-        <visual>
-            <origin xyz="0 -0.075 0" rpy="1.5708 0 0"/>
-            <geometry>
-                <cylinder radius="${needle_radius}" length = "${needle_length}" />
-            </geometry>
-            <material name="blue"/>
-        </visual>
-    </link-->
-<xacro:property name="link_qty" value="2"/>
-<xacro:property name="link_length" value="${needle_length/ link_qty}"/>
-<xacro:property name="link_radius" value="${needle_radius}"/>
-<xacro:property name="link_mass" value="0.01"/>
-<xacro:property name="needle_radius" value="0.001" />
-<xacro:property name="needle_length" value="0.15" />
-<!-- Macro pour un maillon du serpent -->
-<xacro:macro name="needle_link" params="id">
-    <link name="link_${id}">
-        <visual>
-            <geometry>
-                <cylinder length="${link_length}" radius="${link_radius}"/>
-            </geometry>
-            <material name="blue"/>
-            <origin xyz="0 -0.075 0" rpy="0 1.5708 1.5708"/>
-        </visual>
-    </link>
-    <!-- Joint to connect to the root link or previous link -->
-    <xacro:if value="${id == 1}">
-            <joint name="joint_needle" type="prismatic">
-            <parent link="link_y"/>
-            <child link="link_${id}"/>
-            <origin xyz="0 0 ${link_y_size_z/2}" rpy="0 0 0"/>
-            <axis xyz="0 1 0"/>
-            <limit effort="1000" velocity="0.5" lower="${link_y_size_y}" upper="-0.04"/>
-        </joint>
-    </xacro:if>
-    <xacro:unless value="${id == 1}">
-        <joint name="joint_${id-1}_${id}" type="revolute">
-            <parent link="link_${id-1}"/>
-            <child link="link_${id}"/>
-            <origin xyz="0 ${link_length} 0" rpy="0 0 0"/>
-            <axis xyz="0 0 1"/>
-            <limit effort="30" velocity="0.5" lower="-${needle_radius * 70}" upper="${needle_radius * 70}"/>
-        </joint>
-    </xacro:unless>
-</xacro:macro>
-<xacro:macro name="generate_links" params="current_link max_link">
-    <xacro:needle_link id="${current_link}"/>
-    <xacro:if value="${current_link != max_link}">
-        <xacro:generate_links current_link="${current_link + 1}" max_link="${max_link}"/>
-    </xacro:if>
-</xacro:macro>
-<xacro:generate_links current_link="1" max_link="${link_qty}"/>
 </robot>
